Commit message: feat: add grippers, gripper_viz node and data recorder

File: src/dual_arm_description/urdf/dual_ur5e.urdf.xacro (robot description, xacro)
@@ -2,4 +2,5 @@
 <robot xmlns:xacro="http://www.ros.org/wiki/xacro" name="dual_ur5e">
   <xacro:include filename="$(find ur_description)/urdf/ur_macro.xacro"/>
+  <xacro:include filename="$(find dual_arm_description)/urdf/robotiq_2f_85_macro.xacro"/>
   <!-- Root -->
   <link name="world"/>
@@ -55,3 +56,11 @@
     <origin xyz="0 -0.5 0.025" rpy="0 0 0"/>
   </xacro:ur_robot>
+  <!-- LEFT gripper attached to left_tool0 -->
+  <xacro:robotiq_2f_85 prefix="left_" parent="left_tool0">
+    <origin xyz="0 0 0" rpy="0 0 0"/>
+  </xacro:robotiq_2f_85>
+  <!-- RIGHT gripper attached to right_tool0 -->
+  <xacro:robotiq_2f_85 prefix="right_" parent="right_tool0">
+    <origin xyz="0 0 0" rpy="0 0 0"/>
+  </xacro:robotiq_2f_85>
 </robot>
